Commit message: rotation of ee_link fixed

File: tams_ur5_description/urdf/ur5.urdf.xacro (robot description, xacro)
@@ -1,44 +1,42 @@
 <?xml version="1.0"?>
 <robot xmlns:xacro="http://wiki.ros.org/xacro" name="ur5_robot">
- <xacro:macro name="ur5_robot"
-               params="
-                 prefix
-                 joint_limit_params
-                 kinematics_params
-                 transmission_hw_interface
-               ">
-  <!-- specify which robot loaded by ur_macro.xacro -->
-  <xacro:arg name="robot_model" default="ur5"/>
-  <!--ur5 parameters files -->
-  <xacro:property name="physical_params" value="$(find ur_description)/config/ur5/physical_parameters.yaml"/>
-  <xacro:property name="visual_params" value="$(find ur_description)/config/ur5/visual_parameters.yaml"/>
-  <!--common parameters -->
-  <!-- If True, enable the safety limits controller -->
-  <xacro:property name="safety_limits" value="false"/>
-  <!-- The lower/upper limits in the safety controller -->
-  <xacro:property name="safety_pos_margin" value="0.15" />
-  <!-- Used to set k position in the safety controller -->
-  <xacro:property name="safety_k_position" value="20" />
-   <!-- import main macro -->
-   <xacro:include filename="$(find ur_description)/urdf/inc/ur_macro.xacro"/>
-   <!-- arm -->
-   <xacro:ur_robot
-     prefix="${prefix}"
-     joint_limits_parameters_file="${joint_limit_params}"
-     kinematics_parameters_file="${kinematics_params}"
-     physical_parameters_file="${physical_params}"
-     visual_parameters_file="${visual_params}"
-     transmission_hw_interface="${transmission_hw_interface}"
-     safety_limits="${safety_limits}"
-     safety_pos_margin="${safety_pos_margin}"
-     safety_k_position="${safety_k_position}"/>
-  <xacro:include filename="$(find tams_ur5_setup_description)/urdf/upstream/ur.gazebo.xacro" />
-  <xacro:ur_arm_gazebo prefix="${prefix}" />
-  <joint name="${prefix}ee_fixed_joint" type="fixed">
-      <parent link="${prefix}flange" />
-      <child link = "${prefix}ee_link" />
-      <origin xyz="0.0 0.0 0.0" rpy="${pi/2.0} 0.0 0.0" />
-    </joint>
-    <link name="${prefix}ee_link"/>
- </xacro:macro>
+    <xacro:macro name="ur5_robot"
+        params="
+        prefix
+        joint_limit_params
+        kinematics_params
+        transmission_hw_interface
+        ">
+        <!--ur5 parameters files -->
+        <xacro:property name="physical_params" value="$(find ur_description)/config/ur5/physical_parameters.yaml"/>
+        <xacro:property name="visual_params" value="$(find ur_description)/config/ur5/visual_parameters.yaml"/>
+        <!--common parameters -->
+        <!-- If True, enable the safety limits controller -->
+        <xacro:property name="safety_limits" value="false"/>
+        <!-- The lower/upper limits in the safety controller -->
+        <xacro:property name="safety_pos_margin" value="0.15" />
+        <!-- Used to set k position in the safety controller -->
+        <xacro:property name="safety_k_position" value="20" />
+        <!-- import main macro -->
+        <xacro:include filename="$(find ur_description)/urdf/inc/ur_macro.xacro"/>
+        <!-- arm -->
+        <xacro:ur_robot
+            prefix="${prefix}"
+            joint_limits_parameters_file="${joint_limit_params}"
+            kinematics_parameters_file="${kinematics_params}"
+            physical_parameters_file="${physical_params}"
+            visual_parameters_file="${visual_params}"
+            transmission_hw_interface="${transmission_hw_interface}"
+            safety_limits="${safety_limits}"
+            safety_pos_margin="${safety_pos_margin}"
+            safety_k_position="${safety_k_position}"/>
+        <xacro:include filename="$(find tams_ur5_setup_description)/urdf/upstream/ur.gazebo.xacro" />
+        <xacro:ur_arm_gazebo prefix="${prefix}" />
+        <joint name="${prefix}ee_fixed_joint" type="fixed">
+            <parent link="${prefix}flange" />
+            <child link = "${prefix}ee_link" />
+            <origin xyz="0.0 0.0 0.0" rpy="${pi} 0.0 0.0" />
+        </joint>
+        <link name="${prefix}ee_link"/>
+    </xacro:macro>
 </robot>
