Commit message: integration of official ROS ur_description package

File: tams_ur5_description/urdf/arm.urdf.xacro (robot description, xacro)
@@ -2,4 +2,8 @@
 <robot xmlns:xacro="http://www.ros.org/wiki/xacro"
        name="arm" >
+  <xacro:arg name="joint_limit_params" default="$(find tams_ur5_description)/config/joint_ranges/default.yaml"/>
+  <xacro:arg name="kinematics_params" default="$(find tams_ur5_description)/config/tams_ur5_calibration.yaml"/>
+  <xacro:arg name="transmission_hw_interface" default="hardware_interface/PositionJointInterface"/>
+  <xacro:property name="flange_link_name" value="ur5_ee_link"/>
   <!-- include macro definitions -->
   <xacro:include filename="$(find tams_ur5_description)/urdf/ur5.urdf.xacro" />
@@ -9,14 +13,13 @@
   <xacro:include filename="$(find tams_ur5_description)/urdf/s_model_adapter.urdf.xacro" />
   <xacro:include filename="$(find tams_ur5_description)/urdf/plug_collision_model.urdf.xacro" />
-  <!-- arm -->
-  <!-- xamla_cap is a custom parameter in TAMS' fork of the universal_robot repository,
-       remove it if you want to use the upstream ur5 description instead -->
-  <xacro:ur5_robot prefix="ur5_" joint_limited="false" xamla_cap="true"/>
+  <!-- ur5 arm -->
+  <xacro:ur5_robot prefix="ur5_" joint_limit_params="$(arg joint_limit_params)"
+                   kinematics_params="$(arg kinematics_params)" transmission_hw_interface="$(arg transmission_hw_interface)"/>
   <!-- ft_adapter -->
-  <xacro:ft_adapter name="ft_adapter" parent="ur5_ee_link">
+  <xacro:ft_adapter name="ft_adapter" parent="${flange_link_name}">
     <origin xyz="0.0045 0.0 0.0" rpy="0.0 ${pi/2} 0.0" />
   </xacro:ft_adapter>
   <!-- ft150 -->
-  <xacro:robotiq_fts150 prefix="ft_" parent="ur5_ee_link">
+  <xacro:robotiq_fts150 prefix="ft_" parent="${flange_link_name}">
     <origin xyz="0.009 0.0 0.0" rpy="0.0 ${-pi/2} ${pi}" />
   </xacro:robotiq_fts150>
@@ -40,5 +43,5 @@
   </joint>
   <!-- plug collision model -->
-  <xacro:plug_collision_model name="plug_collision_model" parent="ur5_ee_link" >
+  <xacro:plug_collision_model name="plug_collision_model" parent="${flange_link_name}">
     <origin xyz="0.0 0.0 0.0" rpy="0.0 0.0 0.0" />
   </xacro:plug_collision_model>

File: tams_ur5_description/urdf/ur5.urdf.xacro (robot description, xacro)
@@ -1,331 +1,44 @@
 <?xml version="1.0"?>
-<robot xmlns:xacro="http://ros.org/wiki/xacro">
-  <xacro:include filename="$(find tams_ur5_setup_description)/urdf/upstream/ur.transmission.xacro" />
+<robot xmlns:xacro="http://wiki.ros.org/xacro" name="ur5_robot">
+ <xacro:macro name="ur5_robot"
+               params="
+                 prefix
+                 joint_limit_params
+                 kinematics_params
+                 transmission_hw_interface
+               ">
+  <!-- specify which robot loaded by ur_macro.xacro -->
+  <xacro:arg name="robot_model" default="ur5"/>
+  <!--ur5 parameters files -->
+  <xacro:property name="physical_params" value="$(find ur_description)/config/ur5/physical_parameters.yaml"/>
+  <xacro:property name="visual_params" value="$(find ur_description)/config/ur5/visual_parameters.yaml"/>
+  <!--common parameters -->
+  <!-- If True, enable the safety limits controller -->
+  <xacro:property name="safety_limits" value="false"/>
+  <!-- The lower/upper limits in the safety controller -->
+  <xacro:property name="safety_pos_margin" value="0.15" />
+  <!-- Used to set k position in the safety controller -->
+  <xacro:property name="safety_k_position" value="20" />
+   <!-- import main macro -->
+   <xacro:include filename="$(find ur_description)/urdf/inc/ur_macro.xacro"/>
+   <!-- arm -->
+   <xacro:ur_robot
+     prefix="${prefix}"
+     joint_limits_parameters_file="${joint_limit_params}"
+     kinematics_parameters_file="${kinematics_params}"
+     physical_parameters_file="${physical_params}"
+     visual_parameters_file="${visual_params}"
+     transmission_hw_interface="${transmission_hw_interface}"
+     safety_limits="${safety_limits}"
+     safety_pos_margin="${safety_pos_margin}"
+     safety_k_position="${safety_k_position}"/>
   <xacro:include filename="$(find tams_ur5_setup_description)/urdf/upstream/ur.gazebo.xacro" />
-  <!-- Inertia parameters -->
-  <xacro:property name="base_mass" value="4.0" />  <!-- This mass might be incorrect -->
-  <xacro:property name="shoulder_mass" value="3.7000" />
-  <xacro:property name="upper_arm_mass" value="8.3930" />
-  <xacro:property name="forearm_mass" value="2.2750" />
-  <xacro:property name="wrist_1_mass" value="1.2190" />
-  <xacro:property name="wrist_2_mass" value="1.2190" />
-  <xacro:property name="wrist_3_mass" value="0.1879" />
-  <xacro:property name="shoulder_cog" value="0.0 0.00193 -0.02561" />
-  <xacro:property name="upper_arm_cog" value="0.0 -0.024201 0.2125" />
-  <xacro:property name="forearm_cog" value="0.0 0.0265 0.11993" />
-  <xacro:property name="wrist_1_cog" value="0.0 0.110949 0.01634" />
-  <xacro:property name="wrist_2_cog" value="0.0 0.0018 0.11099" />
-  <xacro:property name="wrist_3_cog" value="0.0 0.001159 0.0" />
-  <!-- Loads the joint ranges configuration of the ur5 -->
-  <xacro:arg name="joint_ranges_config" default="$(find tams_ur5_description)/config/joint_ranges/default.yaml" />
-  <xacro:property name="joint_limits" value="${xacro.load_yaml('$(arg joint_ranges_config)')}"/>
-  <!-- Kinematic model -->
-  <!-- Properties from urcontrol.conf -->
-  <!--
-    DH for UR5:
-    a = [0.00000, -0.42500, -0.39225,  0.00000,  0.00000,  0.0000]
-    d = [0.089159,  0.00000,  0.00000,  0.10915,  0.09465,  0.0823]
-    alpha = [ 1.570796327, 0, 0, 1.570796327, -1.570796327, 0 ]
-    q_home_offset = [0, -1.570796327, 0, -1.570796327, 0, 0]
-    joint_direction = [-1, -1, 1, 1, 1, 1]
-    mass = [3.7000, 8.3930, 2.2750, 1.2190, 1.2190, 0.1879]
-    center_of_mass = [ [0, -0.02561, 0.00193], [0.2125, 0, 0.11336], [0.11993, 0.0, 0.0265], [0, -0.0018, 0.01634], [0, 0.0018,0.01634], [0, 0, -0.001159] ]
-  -->
-  <xacro:property name="ur5_d1" value="0.089159" />
-  <xacro:property name="ur5_a2" value="-0.42500" />
-  <xacro:property name="ur5_a3" value="-0.39225" />
-  <xacro:property name="ur5_d4" value="0.10915" />
-  <xacro:property name="ur5_d5" value="0.09465" />
-  <xacro:property name="ur5_d6" value="0.0823" />
-  <!-- Arbitrary offsets for shoulder/elbow joints -->
-  <xacro:property name="shoulder_offset" value="0.13585" />  <!-- measured from model -->
-  <xacro:property name="elbow_offset" value="-0.1197" /> <!-- measured from model -->
-  <!-- link lengths used in model -->
-  <xacro:property name="shoulder_height" value="${ur5_d1}" />
-  <xacro:property name="upper_arm_length" value="${-ur5_a2}" />
-  <xacro:property name="forearm_length" value="${-ur5_a3}" />
-  <xacro:property name="wrist_1_length" value="${ur5_d4 - elbow_offset - shoulder_offset}" />
-  <xacro:property name="wrist_2_length" value="${ur5_d5}" />
-  <xacro:property name="wrist_3_length" value="${ur5_d6}" />
-  <!--property name="shoulder_height" value="0.089159" /-->
-  <!--property name="shoulder_offset" value="0.13585" /-->  <!-- shoulder_offset - elbow_offset + wrist_1_length = 0.10915 -->
-  <!--property name="upper_arm_length" value="0.42500" /-->
-  <!--property name="elbow_offset" value="0.1197" /-->       <!-- CAD measured -->
-  <!--property name="forearm_length" value="0.39225" /-->
-  <!--property name="wrist_1_length" value="0.093" /-->     <!-- CAD measured -->
-  <!--property name="wrist_2_length" value="0.09465" /-->   <!-- In CAD this distance is 0.930, but in the spec it is 0.09465 -->
-  <!--property name="wrist_3_length" value="0.0823" /-->
-  <xacro:property name="shoulder_radius" value="0.060" />   <!-- manually measured -->
-  <xacro:property name="upper_arm_radius" value="0.054" />  <!-- manually measured -->
-  <xacro:property name="elbow_radius" value="0.060" />      <!-- manually measured -->
-  <xacro:property name="forearm_radius" value="0.040" />    <!-- manually measured -->
-  <xacro:property name="wrist_radius" value="0.045" />      <!-- manually measured -->
-  <xacro:macro name="cylinder_inertial" params="radius length mass *origin">
-    <inertial>
-      <mass value="${mass}" />
-      <xacro:insert_block name="origin" />
-      <inertia ixx="${0.0833333 * mass * (3 * radius * radius + length * length)}" ixy="0.0" ixz="0.0"
-        iyy="${0.0833333 * mass * (3 * radius * radius + length * length)}" iyz="0.0"
-        izz="${0.5 * mass * radius * radius}" />
-    </inertial>
-  </xacro:macro>
-  <!--
-    The parameter xamla_cap enables optional support for Xamla's rounded cap (wrist 2)
-    increasing the collision free space.
-    If set, visual and collision meshes are loaded from the files provided in the following
-    repository: https://github.com/Xamla/xamla_egomo.
-    More information on the cap and the 3D-printable models can be found at:
-    https://github.com/Xamla/xamla_egomo/tree/master/egomo_3d_printed_parts/egomo-1
-  -->
-  <xacro:macro name="ur5_robot" params="prefix joint_limited
-    xamla_cap:=false
-    transmission_hw_interface:=hardware_interface/PositionJointInterface">
-    <link name="${prefix}base_link" >
-      <visual>
-        <geometry>
-          <mesh filename="package://ur_description/meshes/ur5/visual/base.dae" />
-        </geometry>
-        <material name="LightGrey">
-          <color rgba="0.7 0.7 0.7 1.0"/>
-        </material>
-      </visual>
-      <collision>
-        <geometry>
-          <mesh filename="package://ur_description/meshes/ur5/collision/base.stl" />
-        </geometry>
-      </collision>
-      <xacro:cylinder_inertial radius="0.06" length="0.05" mass="${base_mass}">
-        <origin xyz="0.0 0.0 0.0" rpy="0 0 0" />
-      </xacro:cylinder_inertial>
-    </link>
-    <joint name="${prefix}shoulder_pan_joint" type="revolute">
-      <parent link="${prefix}base_link" />
-      <child link = "${prefix}shoulder_link" />
-      <origin xyz="0.0 0.0 ${shoulder_height}" rpy="0.0 0.0 0.0" />
-      <axis xyz="0 0 1" />
-      <xacro:unless value="${joint_limited}">
-        <limit lower="${joint_limits['shoulder_pan_joint']['lower']}" upper="${joint_limits['shoulder_pan_joint']['upper']}" effort="150.0" velocity="3.15"/>
-      </xacro:unless>
-      <xacro:if value="${joint_limited}">
-        <limit lower="${-pi}" upper="${pi}" effort="150.0" velocity="3.15"/>
-      </xacro:if>
-      <dynamics damping="0.0" friction="0.0"/>
+  <xacro:ur_arm_gazebo prefix="${prefix}" />
+  <joint name="${prefix}ee_fixed_joint" type="fixed">
+      <parent link="${prefix}flange" />
+      <child link = "${prefix}ee_link" />
+      <origin xyz="0.0 0.0 0.0" rpy="${pi/2.0} 0.0 0.0" />
     </joint>
-    <link name="${prefix}shoulder_link">
-      <visual>
-        <geometry>
-          <mesh filename="package://ur_description/meshes/ur5/visual/shoulder.dae" />
-        </geometry>
-        <material name="LightGrey">
-          <color rgba="0.7 0.7 0.7 1.0"/>
-        </material>
-      </visual>
-      <collision>
-        <geometry>
-          <mesh filename="package://ur_description/meshes/ur5/collision/shoulder.stl" />
-        </geometry>
-      </collision>
-      <xacro:cylinder_inertial radius="0.06" length="0.15" mass="${shoulder_mass}">
-        <origin xyz="0.0 0.0 0.0" rpy="0 0 0" />
-      </xacro:cylinder_inertial>
-    </link>
-    <joint name="${prefix}shoulder_lift_joint" type="revolute">
-      <parent link="${prefix}shoulder_link" />
-      <child link = "${prefix}upper_arm_link" />
-      <origin xyz="0.0 ${shoulder_offset} 0.0" rpy="0.0 ${pi / 2.0} 0.0" />
-      <axis xyz="0 1 0" />
-      <xacro:unless value="${joint_limited}">
-      	<limit lower="${joint_limits['shoulder_lift_joint']['lower']}" upper="${joint_limits['shoulder_lift_joint']['upper']}" effort="150.0" velocity="3.15"/>
-      </xacro:unless>
-      <xacro:if value="${joint_limited}">
-        <limit lower="${-pi}" upper="${pi}" effort="150.0" velocity="3.15"/>
-      </xacro:if>
-      <dynamics damping="0.0" friction="0.0"/>
-    </joint>
-    <link name="${prefix}upper_arm_link">
-      <visual>
-        <geometry>
-          <mesh filename="package://ur_description/meshes/ur5/visual/upperarm.dae" />
-        </geometry>
-        <material name="LightGrey">
-          <color rgba="0.7 0.7 0.7 1.0"/>
-        </material>
-      </visual>
-      <collision>
-        <geometry>
-          <mesh filename="package://ur_description/meshes/ur5/collision/upperarm.stl" />
-        </geometry>
-      </collision>
-      <xacro:cylinder_inertial radius="0.06" length="0.56" mass="${upper_arm_mass}">
-        <origin xyz="0.0 0.0 0.28" rpy="0 0 0" />
-      </xacro:cylinder_inertial>
-    </link>
-    <joint name="${prefix}elbow_joint" type="revolute">
-      <parent link="${prefix}upper_arm_link" />
-      <child link = "${prefix}forearm_link" />
-      <origin xyz="0.0 ${elbow_offset} ${upper_arm_length}" rpy="0.0 0.0 0.0" />
-      <axis xyz="0 1 0" />
-      <xacro:unless value="${joint_limited}">
-      	<limit lower="${joint_limits['elbow_joint']['lower']}" upper="${joint_limits['elbow_joint']['upper']}" effort="150.0" velocity="3.15"/>
-      </xacro:unless>
-      <xacro:if value="${joint_limited}">
-        <limit lower="${-pi}" upper="${pi}" effort="150.0" velocity="3.15"/>
-      </xacro:if>
-      <dynamics damping="0.0" friction="0.0"/>
-    </joint>
-    <link name="${prefix}forearm_link">
-      <visual>
-        <geometry>
-          <mesh filename="package://ur_description/meshes/ur5/visual/forearm.dae" />
-        </geometry>
-        <material name="LightGrey">
-          <color rgba="0.7 0.7 0.7 1.0"/>
-        </material>
-      </visual>
-      <collision>
-        <geometry>
-          <mesh filename="package://ur_description/meshes/ur5/collision/forearm.stl" />
-        </geometry>
-      </collision>
-      <xacro:cylinder_inertial radius="0.06" length="0.5" mass="${forearm_mass}">
-        <origin xyz="0.0 0.0 0.25" rpy="0 0 0" />
-      </xacro:cylinder_inertial>
-    </link>
-    <joint name="${prefix}wrist_1_joint" type="revolute">
-      <parent link="${prefix}forearm_link" />
-      <child link = "${prefix}wrist_1_link" />
-      <origin xyz="0.0 0.0 ${forearm_length}" rpy="0.0 ${pi / 2.0} 0.0" />
-      <axis xyz="0 1 0" />
-      <xacro:unless value="${joint_limited}">
-      	<limit lower="${joint_limits['wrist_1_joint']['lower']}" upper="${joint_limits['wrist_1_joint']['upper']}" effort="28.0" velocity="3.2"/>
-      </xacro:unless>
-      <xacro:if value="${joint_limited}">
-        <limit lower="${-pi}" upper="${pi}" effort="28.0" velocity="3.2"/>
-      </xacro:if>
-      <dynamics damping="0.0" friction="0.0"/>
-    </joint>
-    <link name="${prefix}wrist_1_link">
-      <visual>
-        <geometry>
-          <mesh filename="package://ur_description/meshes/ur5/visual/wrist1.dae" />
-        </geometry>
-        <material name="LightGrey">
-          <color rgba="0.7 0.7 0.7 1.0"/>
-        </material>
-      </visual>
-      <collision>
-        <geometry>
-          <mesh filename="package://ur_description/meshes/ur5/collision/wrist1.stl" />
-        </geometry>
-      </collision>
-      <xacro:cylinder_inertial radius="0.6" length="0.12" mass="${wrist_1_mass}">
-        <origin xyz="0.0 0.0 0.0" rpy="0 0 0" />
-      </xacro:cylinder_inertial>
-    </link>
-    <joint name="${prefix}wrist_2_joint" type="revolute">
-      <parent link="${prefix}wrist_1_link" />
-      <child link = "${prefix}wrist_2_link" />
-      <origin xyz="0.0 ${wrist_1_length} 0.0" rpy="0.0 0.0 0.0" />
-      <axis xyz="0 0 1" />
-      <xacro:unless value="${joint_limited}">
-	<limit lower="${joint_limits['wrist_2_joint']['lower']}" upper="${joint_limits['wrist_2_joint']['upper']}" effort="28.0" velocity="3.2"/>
-      </xacro:unless>
-      <xacro:if value="${joint_limited}">
-        <limit lower="${-pi}" upper="${pi}" effort="28.0" velocity="3.2"/>
-      </xacro:if>
-      <dynamics damping="0.0" friction="0.0"/>
-    </joint>
-    <link name="${prefix}wrist_2_link">
-      <visual>
-        <geometry>
-          <xacro:if value="${xamla_cap}">
-            <mesh filename="package://tams_ur5_description/meshes/ur5/visual/wrist2_rounded.dae" />
-          </xacro:if>
-          <xacro:unless value="${xamla_cap}">
-            <mesh filename="package://ur_description/meshes/ur5/visual/wrist2.dae" />
-          </xacro:unless>
-        </geometry>
-        <material name="LightGrey">
-          <color rgba="0.7 0.7 0.7 1.0"/>
-        </material>
-      </visual>
-      <collision>
-        <geometry>
-          <xacro:if value="${xamla_cap}">
-            <mesh filename="package://tams_ur5_description/meshes/ur5/collision/wrist2_rounded.stl" />
-          </xacro:if>
-          <xacro:unless value="${xamla_cap}">
-	    <mesh filename="package://ur_description/meshes/ur5/collision/wrist2.stl" />
-          </xacro:unless>
-        </geometry>
-      </collision>
-      <xacro:cylinder_inertial radius="0.6" length="0.12" mass="${wrist_2_mass}">
-        <origin xyz="0.0 0.0 0.0" rpy="0 0 0" />
-      </xacro:cylinder_inertial>
-    </link>
-    <joint name="${prefix}wrist_3_joint" type="revolute">
-      <parent link="${prefix}wrist_2_link" />
-      <child link = "${prefix}wrist_3_link" />
-      <origin xyz="0.0 0.0 ${wrist_2_length}" rpy="0.0 0.0 0.0" />
-      <axis xyz="0 1 0" />
-      <xacro:unless value="${joint_limited}">
-	<limit lower="${joint_limits['wrist_3_joint']['lower']}" upper="${joint_limits['wrist_3_joint']['upper']}" effort="28.0" velocity="3.2"/>
-      </xacro:unless>
-      <xacro:if value="${joint_limited}">
-        <limit lower="${-pi}" upper="${pi}" effort="28.0" velocity="3.2"/>
-      </xacro:if>
-      <dynamics damping="0.0" friction="0.0"/>
-    </joint>
-    <link name="${prefix}wrist_3_link">
-      <visual>
-        <geometry>
-          <mesh filename="package://ur_description/meshes/ur5/visual/wrist3.dae" />
-        </geometry>
-        <material name="LightGrey">
-          <color rgba="0.7 0.7 0.7 1.0"/>
-        </material>
-      </visual>
-      <collision>
-        <geometry>
-          <mesh filename="package://ur_description/meshes/ur5/collision/wrist3.stl" />
-        </geometry>
-      </collision>
-      <xacro:cylinder_inertial radius="0.6" length="0.12" mass="${wrist_3_mass}">
-        <origin xyz="0.0 0.0 0.0" rpy="0 0 0" />
-      </xacro:cylinder_inertial>
-    </link>
-    <joint name="${prefix}ee_fixed_joint" type="fixed">
-      <parent link="${prefix}wrist_3_link" />
-      <child link = "${prefix}ee_link" />
-      <origin xyz="0.0 ${wrist_3_length} 0.0" rpy="0.0 0.0 ${pi/2.0}" />
-    </joint>
-    <link name="${prefix}ee_link">
-      <collision>
-        <geometry>
-          <box size="0.01 0.01 0.01"/>
-        </geometry>
-        <origin rpy="0 0 0" xyz="-0.01 0 0"/>
-      </collision>
-    </link>
-    <xacro:ur_arm_transmission prefix="${prefix}"/>
-    <xacro:ur_arm_gazebo prefix="${prefix}" />
-    <!-- ROS base_link to UR 'Base' Coordinates transform -->
-    <link name="${prefix}base"/>
-    <joint name="${prefix}base_link-base_fixed_joint" type="fixed">
-      <!-- NOTE: this rotation is only needed as long as base_link itself is
-                 not corrected wrt the real robot (ie: rotated over 180
-                 degrees)
-      -->
-      <origin xyz="0 0 0" rpy="0 0 ${-pi}"/>
-      <parent link="${prefix}base_link"/>
-      <child link="${prefix}base"/>
-    </joint>
-    <!-- Frame coincident with all-zeros TCP on UR controller -->
-    <link name="${prefix}tool0"/>
-    <joint name="${prefix}wrist_3_link-tool0_fixed_joint" type="fixed">
-      <origin xyz="0 ${wrist_3_length} 0" rpy="${pi/-2.0} 0 0"/>
-      <parent link="${prefix}wrist_3_link"/>
-      <child link="${prefix}tool0"/>
-    </joint>
-  </xacro:macro>
+    <link name="${prefix}ee_link"/>
+ </xacro:macro>
 </robot>

Commit message: improved integration of ur5 ur_description

File: tams_ur5_description/urdf/arm.urdf.xacro (robot description, xacro)
@@ -2,10 +2,10 @@
 <robot xmlns:xacro="http://www.ros.org/wiki/xacro"
        name="arm" >
-  <xacro:arg name="joint_limit_params" default="$(find tams_ur5_description)/config/joint_ranges/default.yaml"/>
-  <xacro:arg name="kinematics_params" default="$(find tams_ur5_description)/config/tams_ur5_calibration.yaml"/>
+  <xacro:arg name="ur5_prefix" default="ur5_"/>
+  <xacro:arg name="joint_limits_parameters_file" default="$(find tams_ur5_description)/config/joint_ranges/default.yaml"/>
+  <xacro:arg name="kinematics_parameters_file" default="$(find tams_ur5_description)/config/tams_ur5_calibration.yaml"/>
   <xacro:arg name="transmission_hw_interface" default="hardware_interface/PositionJointInterface"/>
-  <xacro:property name="flange_link_name" value="ur5_ee_link"/>
   <!-- include macro definitions -->
-  <xacro:include filename="$(find tams_ur5_description)/urdf/ur5.urdf.xacro" />
+  <xacro:include filename="$(find ur_description)/urdf/inc/ur5_macro.xacro"/>
   <xacro:include filename="$(find robotiq_3f_gripper_visualization)/cfg/robotiq-3f-gripper_articulated_macro.xacro"/>
   <xacro:include filename="$(find robotiq_ft_sensor)/urdf/robotiq_fts150.urdf.xacro" />
@@ -14,6 +14,18 @@
   <xacro:include filename="$(find tams_ur5_description)/urdf/plug_collision_model.urdf.xacro" />
   <!-- ur5 arm -->
-  <xacro:ur5_robot prefix="ur5_" joint_limit_params="$(arg joint_limit_params)"
-                   kinematics_params="$(arg kinematics_params)" transmission_hw_interface="$(arg transmission_hw_interface)"/>
+  <xacro:ur5_robot prefix="$(arg ur5_prefix)" joint_limits_parameters_file="$(arg joint_limits_parameters_file)"
+                   kinematics_parameters_file="$(arg kinematics_parameters_file)" transmission_hw_interface="$(arg transmission_hw_interface)"/>
+  <!-- gazebo params for ur5 -->
+  <xacro:include filename="$(find tams_ur5_setup_description)/urdf/upstream/ur.gazebo.xacro" />
+  <xacro:ur_arm_gazebo prefix="$(arg ur5_prefix)" />
+  <!-- link which was used on previous tams_ur5_description to attach tools -->
+  <link name="$(arg ur5_prefix)ee_link"/>
+  <joint name="$(arg ur5_prefix)ee_fixed_joint" type="fixed">
+      <parent link="$(arg ur5_prefix)flange" />
+      <child link ="$(arg ur5_prefix)ee_link" />
+      <origin xyz="0.0 0.0 0.0" rpy="${pi} 0.0 0.0" />
+  </joint>
+  <!-- <xacro:property name="flange_link_name" value="${prefix}flange}"/> -->
+  <xacro:property name="flange_link_name" value="$(arg ur5_prefix)ee_link"/>
   <!-- ft_adapter -->
   <xacro:ft_adapter name="ft_adapter" parent="${flange_link_name}">
